Commit message: Add files for simulation in Gazebo

File: catkin_ws/src/chefbot_description/urdf/chefbot.xacro (robot description, xacro)
@@ -1,5 +1,4 @@
 <?xml version="1.0"?>
 <robot name="chefbot" xmlns:xacro="http://ros.org/wiki/xacro">
-<!--   <xacro:macro name="qbo">   -->
   <xacro:include filename="$(find chefbot_description)/urdf/common_properties.xacro" />
   <xacro:include filename="$(find chefbot_description)/gazebo/chefbot.gazebo.xacro" />
